File: TriCon.kicad_pcb (KiCad board)
At the start: 2 copper layers, 27.3 x 30.3 mm, 14 parts, among them J1 STM32 Debug, SW1 SW_SPDT, U1 STM32F303K8T6

Commit message: 基板 V1.1
Parts:
- Center Controller: renamed from Controller Center
- Left Controller: renamed from Controller Left
- Right Controller: renamed from Controller Right
- renumbered CR2032 to BT1
Connections:
- U1 pad 28: Net-(J2-Pad3) -> Net-(J3-Pad4)
- U1 pad 29: Net-(J2-Pad4) -> Net-(J2-Pad3)
- U1 pad 30: Net-(J3-Pad4) -> Net-(J2-Pad4)
Routing:
- net Net-(J3-Pad4): track 18.7 -> 20.6 mm
- net Net-(J2-Pad4): track 12.9 -> 14.0 mm
- net Net-(J2-Pad3): track 8.09 -> 9.17 mm
Other:
- board text added: "+"
- board text added: "-"
- board text added: "TriCon v1.1"
