File: TriCon.sch (KiCad schematic (older format))
At the start: 14 parts, among them J1 STM32 Debug, J2 OLED128x64, J3 Controller Left, J4 Controller Right, J5 Controller Center, SW1 SW_SPDT, U1 STM32F303K8T6

Commit message: 基板 V1.1
Connections:
- net at J3.4 (SW_D): now also U1.28 (PB5); no longer U1.30 (PB7)
- net at J2.3 (SCL): now also U1.29 (PB6); no longer U1.28 (PB5)
- net at J2.4 (SDA): now also U1.30 (PB7); no longer U1.29 (PB6)
Changed lines of the file:
@@
 Sheet 1 1
 Title "Tri Con"
-Date "2020-04-26"
-Rev "1.0"
+Date "2020-06-16"
+Rev "1.1"
 Comp ""
 Comment1 ""
@@
 	3450 3550 3750 3550
 Wire Wire Line
-	3750 3550 3750 2500
-Wire Wire Line
-	5100 2500 5100 2800
-Wire Wire Line
 	3450 3650 3850 3650
 Wire Wire Line
@@
 	6750 3650 6950 3650
 Wire Wire Line
-	3750 2500 5100 2500
-Wire Wire Line
 	3450 3150 3650 3150
 Wire Wire Line
-	6550 2600 5200 2600
-Wire Wire Line
-	5200 2600 5200 2800
-Wire Wire Line
-	5300 2500 5300 2800
-Wire Wire Line
-	5300 2500 6550 2500
+	5100 2600 5100 2800
+Wire Wire Line
+	5200 2500 5200 2800
 $Comp
 L power:+3V0 #PWR05
@@
 Connection ~ 8750 1650
 Connection ~ 8750 1950
+Wire Wire Line
+	3750 2400 3750 3550
+Wire Wire Line
+	5100 2600 6550 2600
+Wire Wire Line
+	5200 2500 6550 2500
+Wire Wire Line
+	5300 2400 5300 2800
+Wire Wire Line
+	3750 2400 5300 2400
 $EndSCHEMATC
